File: v1/5940.brd (EAGLE design)
At the start: 97.5 x 74.9 mm, 48 parts, among them Q1 IRF540, Q2 IRF540, Q3 IRF540, Q4 IRF540, Q5 IRF540, Q6 IRF540, Q7 IRF540, Q8 IRF540, U1 TLC5940-NT

Commit message: Minor updates
Parts:
- removed 8-15: (no value), SparkFun-Connectors:1X08_LONGPADS
- added JP1: (no value), SparkFun-Connectors:1X08_ROUND
Connections:
- net IN10: now also JP1.3; no longer 8-15.3
- net IN11: now also JP1.4; no longer 8-15.4
- net IN12: now also JP1.5; no longer 8-15.5
- net IN13: now also JP1.6; no longer 8-15.6
- net IN14: now also JP1.7; no longer 8-15.7
- net IN15: now also JP1.8; no longer 8-15.8
- net IN8: now also JP1.1; no longer 8-15.1
- net IN9: now also JP1.2; no longer 8-15.2
Routing:
- net IN9: track 3.81 -> 3.17 mm
- net IN8: track 3.81 -> 3.17 mm
- net IN15: track 12.5 -> 11.8 mm
- net IN14: track 3.81 -> 3.17 mm
- net IN13: track 3.81 -> 3.17 mm
- net IN12: track 3.81 -> 3.17 mm
- net IN11: track 3.81 -> 3.17 mm
- net IN10: track 3.81 -> 3.17 mm
- added copper zone on layer 16, net GND
- removed copper zone on layer 16, net N$17
Changed lines of the file:
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@@
 <element name="TLC_IN_1" library="SparkFun-Connectors" package="SCREWTERMINAL-5MM-2" value="M025MM" x="39.22" y="68.81"/>
 <element name="TLC_OUT" library="SparkFun-Connectors" package="SCREWTERMINAL-5MM-2" value="M025MM" x="59.22" y="68.81"/>
-<element name="8-15" library="SparkFun-Connectors" package="1X08_LONGPADS" value="" x="57.15" y="48.895"/>
 <element name="POWER" library="SparkFun-Connectors" package="1X03_LONGPADS" value="" x="12.7" y="62.23"/>
+<element name="JP1" library="SparkFun-Connectors" package="1X08_ROUND" value="" x="57.15" y="49.53"/>
 </elements>
 <signals>
@@
 <contactref element="POWER" pad="2"/>
 <contactref element="U1" pad="19"/>
+<polygon width="0.6096" layer="16">
+<vertex x="0" y="0"/>
+<vertex x="0" y="74.93"/>
+<vertex x="97.79" y="74.93"/>
+<vertex x="97.79" y="0"/>
+</polygon>
+<via x="69.85" y="57.15" extent="1-16" drill="1.016" diameter="1.6764" shape="square"/>
+<via x="7.62" y="67.31" extent="1-16" drill="1.016" diameter="1.6764" shape="square"/>
+<via x="17.78" y="41.91" extent="1-16" drill="1.016" diameter="1.6764" shape="square"/>
+<via x="10.16" y="3.81" extent="1-16" drill="1.016" diameter="1.6764" shape="square"/>
 </signal>
 <signal name="5V">
@@
 <signal name="IN8">
 <contactref element="U1" pad="8"/>
-<contactref element="8-15" pad="1"/>
-<wire x1="57.15" y1="48.895" x2="57.15" y2="52.705" width="0.6096" layer="16"/>
+<contactref element="JP1" pad="1"/>
+<wire x1="57.15" y1="49.53" x2="57.15" y2="52.705" width="0.6096" layer="16"/>
 </signal>
 <signal name="IN9">
 <contactref element="U1" pad="9"/>
-<contactref element="8-15" pad="2"/>
-<wire x1="59.69" y1="52.705" x2="59.69" y2="48.895" width="0.6096" layer="16"/>
+<contactref element="JP1" pad="2"/>
+<wire x1="59.69" y1="52.705" x2="59.69" y2="49.53" width="0.6096" layer="16"/>
 </signal>
 <signal name="IN10">
 <contactref element="U1" pad="10"/>
-<contactref element="8-15" pad="3"/>
-<wire x1="62.23" y1="48.895" x2="62.23" y2="52.705" width="0.6096" layer="16"/>
+<contactref element="JP1" pad="3"/>
+<wire x1="62.23" y1="49.53" x2="62.23" y2="52.705" width="0.6096" layer="16"/>
 </signal>
 <signal name="IN11">
 <contactref element="U1" pad="11"/>
-<contactref element="8-15" pad="4"/>
-<wire x1="64.77" y1="52.705" x2="64.77" y2="48.895" width="0.6096" layer="16"/>
+<contactref element="JP1" pad="4"/>
+<wire x1="64.77" y1="52.705" x2="64.77" y2="49.53" width="0.6096" layer="16"/>
 </signal>
 <signal name="IN12">
 <contactref element="U1" pad="12"/>
-<contactref element="8-15" pad="5"/>
-<wire x1="67.31" y1="48.895" x2="67.31" y2="52.705" width="0.6096" layer="16"/>
+<contactref element="JP1" pad="5"/>
+<wire x1="67.31" y1="49.53" x2="67.31" y2="52.705" width="0.6096" layer="16"/>
 </signal>
 <signal name="IN13">
 <contactref element="U1" pad="13"/>
-<contactref element="8-15" pad="6"/>
-<wire x1="69.85" y1="52.705" x2="69.85" y2="48.895" width="0.6096" layer="16"/>
+<contactref element="JP1" pad="6"/>
+<wire x1="69.85" y1="52.705" x2="69.85" y2="49.53" width="0.6096" layer="16"/>
 </signal>
 <signal name="IN14">
 <contactref element="U1" pad="14"/>
-<contactref element="8-15" pad="7"/>
-<wire x1="72.39" y1="48.895" x2="72.39" y2="52.705" width="0.6096" layer="16"/>
+<contactref element="JP1" pad="7"/>
+<wire x1="72.39" y1="49.53" x2="72.39" y2="52.705" width="0.6096" layer="16"/>
 </signal>
 <signal name="IN15">
 <contactref element="U1" pad="15"/>
-<contactref element="8-15" pad="8"/>
-<wire x1="74.93" y1="48.895" x2="74.93" y2="57.785" width="0.6096" layer="16"/>
 <wire x1="74.93" y1="57.785" x2="72.39" y2="60.325" width="0.6096" layer="16"/>
+<contactref element="JP1" pad="8"/>
+<wire x1="74.93" y1="57.785" x2="74.93" y2="49.53" width="0.6096" layer="16"/>
 </signal>
 <signal name="IN0">
@@
 <wire x1="52.07" y1="66.66" x2="54.22" y2="68.81" width="0.6096" layer="16"/>
 </signal>
-<signal name="N$17">
-<polygon width="0.6096" layer="16">
-<vertex x="0" y="0"/>
-<vertex x="0" y="74.93"/>
-<vertex x="97.79" y="74.93"/>
-<vertex x="97.79" y="0"/>
-</polygon>
-</signal>
 </signals>
