File: v1/5940.sch (EAGLE design)
At the start: 48 parts, among them Q1 IRF540, Q2 IRF540, Q3 IRF540, Q4 IRF540, Q5 IRF540, Q6 IRF540, Q7 IRF540, Q8 IRF540, U1 TLC5940-NT

Commit message: Minor updates
Parts:
- removed 8-15: (no value), SparkFun-Connectors:M08LONGPADS
- added JP1: (no value), SparkFun-Connectors:M08
Connections:
- net IN10: now also JP1.3; no longer 8-15.3
- net IN11: now also JP1.4; no longer 8-15.4
- net IN12: now also JP1.5; no longer 8-15.5
- net IN13: now also JP1.6; no longer 8-15.6
- net IN14: now also JP1.7; no longer 8-15.7
- net IN15: now also JP1.8; no longer 8-15.8
- net IN8: now also JP1.1; no longer 8-15.1
- net IN9: now also JP1.2; no longer 8-15.2
Changed lines of the file:
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@@
 <part name="TLC_IN_1" library="SparkFun-Connectors" deviceset="M02" device="5MM"/>
 <part name="TLC_OUT" library="SparkFun-Connectors" deviceset="M02" device="5MM"/>
-<part name="8-15" library="SparkFun-Connectors" deviceset="M08" device="LONGPADS"/>
 <part name="POWER" library="SparkFun-Connectors" deviceset="M03" device="LONGPADS"/>
+<part name="JP1" library="SparkFun-Connectors" deviceset="M08" device=""/>
 </parts>
 <sheets>
@@
 <instance part="TLC_IN_1" gate="G$1" x="276.86" y="243.84"/>
 <instance part="TLC_OUT" gate="G$1" x="276.86" y="200.66"/>
-<instance part="8-15" gate="G$1" x="279.4" y="274.32"/>
 <instance part="POWER" gate="G$1" x="223.52" y="276.86"/>
+<instance part="JP1" gate="G$1" x="279.4" y="274.32"/>
 </instances>
 <busses>
@@
 <wire x1="284.48" y1="266.7" x2="294.64" y2="266.7" width="0.1524" layer="91"/>
 <label x="289.56" y="266.7" size="1.778" layer="95"/>
-<pinref part="8-15" gate="G$1" pin="1"/>
+<pinref part="JP1" gate="G$1" pin="1"/>
 </segment>
 </net>
@@
 <wire x1="284.48" y1="269.24" x2="294.64" y2="269.24" width="0.1524" layer="91"/>
 <label x="289.56" y="269.24" size="1.778" layer="95"/>
-<pinref part="8-15" gate="G$1" pin="2"/>
+<pinref part="JP1" gate="G$1" pin="2"/>
 </segment>
 </net>
@@
 <wire x1="284.48" y1="271.78" x2="294.64" y2="271.78" width="0.1524" layer="91"/>
 <label x="289.56" y="271.78" size="1.778" layer="95"/>
-<pinref part="8-15" gate="G$1" pin="3"/>
+<pinref part="JP1" gate="G$1" pin="3"/>
 </segment>
 </net>
@@
 <wire x1="284.48" y1="274.32" x2="294.64" y2="274.32" width="0.1524" layer="91"/>
 <label x="289.56" y="274.32" size="1.778" layer="95"/>
-<pinref part="8-15" gate="G$1" pin="4"/>
+<pinref part="JP1" gate="G$1" pin="4"/>
 </segment>
 </net>
@@
 <wire x1="284.48" y1="276.86" x2="294.64" y2="276.86" width="0.1524" layer="91"/>
 <label x="289.56" y="276.86" size="1.778" layer="95"/>
-<pinref part="8-15" gate="G$1" pin="5"/>
+<pinref part="JP1" gate="G$1" pin="5"/>
 </segment>
 </net>
@@
 <wire x1="284.48" y1="279.4" x2="294.64" y2="279.4" width="0.1524" layer="91"/>
 <label x="289.56" y="279.4" size="1.778" layer="95"/>
-<pinref part="8-15" gate="G$1" pin="6"/>
+<pinref part="JP1" gate="G$1" pin="6"/>
 </segment>
 </net>
@@
 <wire x1="284.48" y1="281.94" x2="294.64" y2="281.94" width="0.1524" layer="91"/>
 <label x="289.56" y="281.94" size="1.778" layer="95"/>
-<pinref part="8-15" gate="G$1" pin="7"/>
+<pinref part="JP1" gate="G$1" pin="7"/>
 </segment>
 </net>
@@
 <wire x1="284.48" y1="284.48" x2="294.64" y2="284.48" width="0.1524" layer="91"/>
 <label x="289.56" y="284.48" size="1.778" layer="95"/>
-<pinref part="8-15" gate="G$1" pin="8"/>
-</segment>
-</net>
+<pinref part="JP1" gate="G$1" pin="8"/>
+</segment>
+</net>
